Commit message: added pendulum controller

File: urdf/inverted_pendulum.xacro (robot description, xacro)
@@ -1,2 +1,3 @@
+this is my first version of inverted pendulum
 <?xml version="1.0"?>
 <robot name="inverted_pendulum" xmlns:xacro="http://ros.org/wiki/xacro">
@@ -49,16 +50,24 @@
   <!-- mark left front wheel as red for orientation -->
   <material>Gazebo/Red</material>
+  <mu1>100</mu1>
+  <mu2>50</mu2>
 </gazebo>
 <xacro:vehicle_wheel link_name="left_rear_wheel" />
 <gazebo reference="left_rear_wheel">
   <material>Gazebo/Grey</material>
+  <mu1>100</mu1>
+  <mu2>50</mu2>
 </gazebo>
 <xacro:vehicle_wheel link_name="right_front_wheel" />
 <gazebo reference="right_front_wheel">
   <material>Gazebo/Grey</material>
+  <mu1>100</mu1>
+  <mu2>50</mu2>
 </gazebo>
 <xacro:vehicle_wheel link_name="right_rear_wheel" />
 <gazebo reference="right_rear_wheel">
   <material>Gazebo/Grey</material>
+  <mu1>100</mu1>
+  <mu2>50</mu2>
 </gazebo>
 <!-- four wheel joints -->
@@ -90,5 +99,5 @@
 <link name="pendulum">
   <inertial>
-    <mass value="1.0" />
+    <mass value="0.1" />
     <origin xyz="0 0 ${pendulum_length/2}" />
     <inertia ixx="0.005" ixy="0.0" ixz="0.0"

Commit message: add one simplified inverted pendulum

File: urdf/inverted_pendulum.xacro (robot description, xacro)
@@ -1,27 +1,9 @@
-this is my first version of inverted pendulum
+<!-- this is a simplified version of inverted pendulum from inverted_pendulum_w_wheels
+without wheels and with linear joint -->
 <?xml version="1.0"?>
 <robot name="inverted_pendulum" xmlns:xacro="http://ros.org/wiki/xacro">
 <xacro:property name="M_PI" value="3.14159265" />
 <xacro:property name="pendulum_length" value="0.3" />
-<xacro:macro name="vehicle_wheel" params="link_name">
-  <link name="${link_name}">
-    <inertial>
-      <mass value="0.1" />
-      <inertia ixx="0.001" ixy="0.0" ixz="0.0"
-        iyy="0.001" iyz="0.0"
-        izz="0.001" />
-    </inertial>
-    <visual>
-      <geometry>
-        <cylinder radius="0.02" length="0.005" />
-      </geometry>
-    </visual>
-    <collision>
-      <geometry>
-        <cylinder radius="0.02" length="0.005" />
-      </geometry>
-    </collision>
-  </link>
-</xacro:macro>
+<link name="world"/>
 <link name="vehicle_body">
   <inertial>
@@ -45,54 +27,10 @@
   <material>Gazebo/Grey</material>
 </gazebo>
-<!-- four wheel links -->
-<xacro:vehicle_wheel link_name="left_front_wheel" />
-<gazebo reference="left_front_wheel">
-  <!-- mark left front wheel as red for orientation -->
-  <material>Gazebo/Red</material>
-  <mu1>100</mu1>
-  <mu2>50</mu2>
-</gazebo>
-<xacro:vehicle_wheel link_name="left_rear_wheel" />
-<gazebo reference="left_rear_wheel">
-  <material>Gazebo/Grey</material>
-  <mu1>100</mu1>
-  <mu2>50</mu2>
-</gazebo>
-<xacro:vehicle_wheel link_name="right_front_wheel" />
-<gazebo reference="right_front_wheel">
-  <material>Gazebo/Grey</material>
-  <mu1>100</mu1>
-  <mu2>50</mu2>
-</gazebo>
-<xacro:vehicle_wheel link_name="right_rear_wheel" />
-<gazebo reference="right_rear_wheel">
-  <material>Gazebo/Grey</material>
-  <mu1>100</mu1>
-  <mu2>50</mu2>
-</gazebo>
-<!-- four wheel joints -->
-<joint name="left_front_joint" type="continuous">
-  <parent link="vehicle_body" />
-  <child link="left_front_wheel" />
-  <origin rpy="${M_PI/2} 0 0" xyz="0.035 0.03 0"/>
-  <axis xyz="0 0 1" />
-</joint>
-<joint name="left_rear_joint" type="continuous">
-  <parent link="vehicle_body" />
-  <child link="left_rear_wheel" />
-  <origin rpy="${M_PI/2} 0 0" xyz="-0.035 0.03 0"/>
-  <axis xyz="0 0 1" />
-</joint>
-<joint name="right_front_joint" type="continuous">
-  <parent link="vehicle_body" />
-  <child link="right_front_wheel" />
-  <origin rpy="${M_PI/2} 0 0" xyz="0.035 -0.03 0"/>
-  <axis xyz="0 0 1" />
-</joint>
-<joint name="right_rear_joint" type="continuous">
-  <parent link="vehicle_body" />
-  <child link="right_rear_wheel" />
-  <origin rpy="${M_PI/2} 0 0" xyz="-0.035 -0.03 0"/>
-  <axis xyz="0 0 1" />
+<joint name="vehicle_joint" type="prismatic">
+  <parent link="world" />
+  <child link="vehicle_body" />
+  <origin xyz="0 0 0.02"/>
+  <axis xyz="1 0 0" />
+  <limit lower="-1" upper="1" effort="10" velocity="10" />
 </joint>
 <!-- the inverted pendulum link -->
@@ -120,8 +58,4 @@
 <gazebo reference="pendulum">
   <material>Gazebo/Blue</material>
-  <!-- <selfCollide>true</selfCollide> -->
-  <!-- why selfCollide is not working with gazebo -->
-  <!-- previous I was trying to use this tag to limit rotation angle by adding two limit blocks, not working -->
-  <gravity>false</gravity>
 </gazebo>
 <!-- the inverted pendulum joint -->

Commit message: add extra mass for pendulum

File: urdf/inverted_pendulum.xacro (robot description, xacro)
@@ -68,3 +68,31 @@
   <!-- set limit for pendulum to not cross vehicle body -->
 </joint>
+<!-- the fixed mass at the top of the pendulum -->
+<link name="pendulum_mass">
+  <inertial>
+    <mass value="1.0" />
+    <inertia ixx="0.001" ixy="0.0" ixz="0.0"
+      iyy="0.001" iyz="0.0"
+      izz="0.001" />
+  </inertial>
+  <visual>
+    <geometry>
+      <sphere radius="0.01" />
+    </geometry>
+  </visual>
+  <collision>
+    <geometry>
+      <sphere radius="0.01" />
+    </geometry>
+  </collision>
+</link>
+<gazebo reference="pendulum_mass">
+  <material>Gazebo/Blue</material>
+</gazebo>
+<!-- fixed joint for pendulum mass -->
+<joint name="pendulum_mass_joint" type="fixed">
+  <parent link="pendulum" />
+  <child link="pendulum_mass" />
+  <origin xyz="0 0 ${pendulum_length}"/>
+</joint>
 </robot>

Commit message: add damping to xacro model

File: urdf/inverted_pendulum.xacro (robot description, xacro)
@@ -32,5 +32,6 @@
   <origin xyz="0 0 0.02"/>
   <axis xyz="1 0 0" />
-  <limit lower="-1" upper="1" effort="10" velocity="10" />
+  <limit lower="-1" upper="1" effort="1000" velocity="1000" />
+  <dynamics damping="0.0" />
 </joint>
 <!-- the inverted pendulum link -->
@@ -65,5 +66,5 @@
   <origin xyz="0 0 0.02"/>
   <axis xyz="0 1 0" />
-  <limit lower="-${M_PI/2}" upper="${M_PI/2}" effort="10" velocity="10" />
+  <limit lower="-${M_PI/2}" upper="${M_PI/2}" effort="1000" velocity="1000" />
   <!-- set limit for pendulum to not cross vehicle body -->
 </joint>
